Commit message: :rewind: Revert urdf changes to fix joint states publish error

File: interbotix_ros_manipulators/interbotix_ros_xsarms/interbotix_xsarm_descriptions/urdf/wx200.urdf.xacro (robot description, xacro)
@@ -1,18 +1,48 @@
 <?xml version="1.0"?>
 <robot name="wx200" xmlns:xacro="http://ros.org/wiki/xacro">
-  <xacro:macro name="boris_arm" params="parent xyz rpy">
-  <xacro:arg name="robot_name" default = "wx200"/>
-  <xacro:arg name="base_link_frame" default="base_link"/>
-  <xacro:arg name="show_ar_tag" default="false"/>
-  <xacro:arg name="show_gripper_bar" default="true"/>
-  <xacro:arg name="show_gripper_fingers" default="true"/>
-  <xacro:arg name="use_world_frame" default="false"/>
-  <xacro:arg name="external_urdf_loc" default=""/>
-  <xacro:arg name="load_gazebo_configs" default="false"/>
-  <xacro:property name="urdf_loc" value="$(arg external_urdf_loc)"/>
-  <xacro:property name="pi_offset" value="0.00001"/>
-  <xacro:if value="$(arg load_gazebo_configs)">
-    <xacro:include filename="$(find interbotix_xsarm_gazebo)/config/interbotix_texture.gazebo"/>
-  </xacro:if>
+  <xacro:property name="robot_model"
+    value="wx200"
+    scope="global"/>
+  <xacro:property name="dof"
+    value="5"
+    scope="global"/>
+  <xacro:arg name="robot_name"                      default="${robot_model}"/>
+  <xacro:arg name="base_link_frame"                 default="base_link"/>
+  <xacro:arg name="use_gripper"                     default="true"/>
+  <xacro:arg name="show_ar_tag"                     default="false"/>
+  <xacro:arg name="show_gripper_bar"                default="true"/>
+  <xacro:arg name="show_gripper_fingers"            default="true"/>
+  <xacro:arg name="use_world_frame"                 default="false"/>
+  <xacro:arg name="external_urdf_loc"               default=""/>
+  <xacro:arg name="hardware_type"                   default="actual"/>
+  <xacro:property name="mesh_directory"             value="package://interbotix_xsarm_descriptions/meshes/${robot_model}_meshes"/>
+  <xacro:property name="urdf_loc"                   value="$(arg external_urdf_loc)"/>
+  <xacro:property name="hardware_type"              value="$(arg hardware_type)"/>
+  <xacro:property name="pi_offset"                  value="0.00001"/>
+  <xacro:property name="waist_limit_effort"         value="8"/>
+  <xacro:property name="waist_limit_lower"          value="${-pi + pi_offset}"/>
+  <xacro:property name="waist_limit_upper"          value="${pi - pi_offset}"/>
+  <xacro:property name="waist_limit_vel"            value="${pi}"/>
+  <xacro:property name="shoulder_limit_effort"      value="18"/>
+  <xacro:property name="shoulder_limit_lower"       value="${radians(-108)}"/>
+  <xacro:property name="shoulder_limit_upper"       value="${radians(113)}"/>
+  <xacro:property name="shoulder_limit_vel"         value="1"/>
+  <xacro:property name="elbow_limit_effort"         value="13"/>
+  <xacro:property name="elbow_limit_lower"          value="${radians(-108)}"/>
+  <xacro:property name="elbow_limit_upper"          value="${radians(93)}"/>
+  <xacro:property name="elbow_limit_vel"            value="${pi}"/>
+  <xacro:property name="wrist_angle_limit_effort"   value="5"/>
+  <xacro:property name="wrist_angle_limit_lower"    value="${radians(-100)}"/>
+  <xacro:property name="wrist_angle_limit_upper"    value="${radians(123)}"/>
+  <xacro:property name="wrist_angle_limit_vel"      value="${pi}"/>
+  <xacro:property name="wrist_rotate_limit_effort"  value="1"/>
+  <xacro:property name="wrist_rotate_limit_lower"   value="${-pi + pi_offset}"/>
+  <xacro:property name="wrist_rotate_limit_upper"   value="${pi - pi_offset}"/>
+  <xacro:property name="wrist_rotate_limit_vel"     value="${pi}"/>
+  <xacro:property name="gripper_limit_vel"          value="${pi}"/>
+  <xacro:property name="finger_limit_effort"        value="5"/>
+  <xacro:property name="finger_limit_lower"         value="0.015"/>
+  <xacro:property name="finger_limit_upper"         value="0.037"/>
+  <xacro:property name="finger_limit_vel"           value="1"/>
   <material name="interbotix_black">
     <texture filename="package://interbotix_xsarm_descriptions/meshes/interbotix_black.png"/>
@@ -21,432 +51,614 @@
     <link name="world"/>
     <joint name="fixed" type="fixed">
-      <parent link="world"/>
-      <child link="$(arg robot_name)/$(arg base_link_frame)"/>
+      <parent
+        link="world"/>
+      <child
+        link="$(arg robot_name)/$(arg base_link_frame)"/>
     </joint>
-  </xacro:if>
-  <joint name="arm_${parent}_joint" type="fixed">
-    <origin xyz="${xyz}" rpy="${rpy}"/>
-    <parent link="${parent}"/>
-    <child link="$(arg robot_name)/$(arg base_link_frame)"/>
-  </joint>
+  </xacro:if> <!-- use_world_frame -->
   <link name="$(arg robot_name)/$(arg base_link_frame)">
     <visual>
-      <origin rpy="0 0 ${pi/2}" xyz="0 0 0"/>
-      <geometry>
-        <mesh filename="package://interbotix_xsarm_descriptions/meshes/wx200_meshes/wx200_1_base.stl" scale="0.001 0.001 0.001"/>
+      <origin
+        rpy="0 0 ${pi/2}"
+        xyz="0 0 0"/>
+      <geometry>
+        <mesh
+          filename="${mesh_directory}/base.stl"
+          scale="0.001 0.001 0.001"/>
       </geometry>
       <material name="interbotix_black"/>
     </visual>
     <collision>
-      <origin rpy="0 0 ${pi/2}" xyz="0 0 0"/>
-      <geometry>
-        <mesh filename="package://interbotix_xsarm_descriptions/meshes/wx200_meshes/wx200_1_base.stl" scale="0.001 0.001 0.001"/>
+      <origin
+        rpy="0 0 ${pi/2}"
+        xyz="0 0 0"/>
+      <geometry>
+        <mesh
+          filename="${mesh_directory}/base.stl"
+          scale="0.001 0.001 0.001"/>
       </geometry>
     </collision>
     <inertial>
-      <origin rpy="0 0 ${pi/2}" xyz="-0.0381747000 0.0006478630 0.0193458000"/>
-      <mass value="0.540142" />
-      <inertia ixx="0.0021190000" iyy="0.0006925000" izz="0.0025280000" ixy="-0.0000172100" ixz="0.0000006389" iyz="0.0000461200" />
+      <origin
+        rpy="0 0 ${pi/2}"
+        xyz="-0.0381747000 0.0006478630 0.0193458000"/>
+      <mass value="0.540142"/>
+      <inertia
+        ixx="0.0021190000"
+        iyy="0.0006925000"
+        izz="0.0025280000"
+        ixy="-0.0000172100"
+        ixz="0.0000006389"
+        iyz="0.0000461200"/>
     </inertial>
   </link>
   <joint name="waist" type="revolute">
     <axis xyz="0 0 1"/>
-    <limit effort="8" lower="${-pi + pi_offset}" upper="${pi - pi_offset}" velocity="${pi}"/>
-    <origin rpy="0 0 0" xyz="0 0 0.072"/>
-    <parent link="$(arg robot_name)/$(arg base_link_frame)"/>
-    <child link="$(arg robot_name)/shoulder_link"/>
-    <dynamics friction="0.1"/>
+    <limit
+      effort="${waist_limit_effort}"
+      lower="${waist_limit_lower}"
+      upper="${waist_limit_upper}"
+      velocity="${waist_limit_vel}"/>
+    <origin
+      rpy="0 0 0"
+      xyz="0 0 0.072"/>
+    <parent
+      link="$(arg robot_name)/$(arg base_link_frame)"/>
+    <child
+      link="$(arg robot_name)/shoulder_link"/>
+    <dynamics
+      friction="0.1"
+      damping="0.1"/>
   </joint>
-  <transmission name="trans_waist">
-    <type>transmission_interface/SimpleTransmission</type>
-    <joint name="waist">
-      <hardwareInterface>hardware_interface/EffortJointInterface</hardwareInterface>
-    </joint>
-    <actuator name="waist_motor">
-      <mechanicalReduction>1</mechanicalReduction>
-    </actuator>
-  </transmission>
   <link name="$(arg robot_name)/shoulder_link">
     <visual>
-      <origin rpy="0 0 ${pi/2}" xyz="0 0 -0.003"/>
-      <geometry>
-        <mesh filename="package://interbotix_xsarm_descriptions/meshes/wx200_meshes/wx200_2_shoulder.stl" scale="0.001 0.001 0.001"/>
+      <origin
+        rpy="0 0 ${pi/2}"
+        xyz="0 0 -0.003"/>
+      <geometry>
+        <mesh
+          filename="${mesh_directory}/shoulder.stl"
+          scale="0.001 0.001 0.001"/>
       </geometry>
       <material name="interbotix_black"/>
     </visual>
     <collision>
-      <origin rpy="0 0 ${pi/2}" xyz="0 0 -0.003"/>
-      <geometry>
-        <mesh filename="package://interbotix_xsarm_descriptions/meshes/wx200_meshes/wx200_2_shoulder.stl" scale="0.001 0.001 0.001"/>
+      <origin
+        rpy="0 0 ${pi/2}"
+        xyz="0 0 -0.003"/>
+      <geometry>
+        <mesh
+          filename="${mesh_directory}/shoulder.stl"
+          scale="0.001 0.001 0.001"/>
       </geometry>
     </collision>
     <inertial>
-      <origin rpy="0 0 ${pi/2}" xyz="0.0000223210 0.0000414608 0.0066287000"/>
-      <mass value="0.480879" />
-      <inertia ixx="0.0003790000" iyy="0.0005557000" izz="0.0005889000" ixy="0.0000000022" ixz="-0.0000003561" iyz="0.0000012247" />
+      <origin
+        rpy="0 0 ${pi/2}"
+        xyz="0.0000223210 0.0000414608 0.0066287000"/>
+      <mass value="0.480879"/>
+      <inertia
+        ixx="0.0003790000"
+        iyy="0.0005557000"
+        izz="0.0005889000"
+        ixy="0.0000000022"
+        ixz="-0.0000003561"
+        iyz="0.0000012247"/>
     </inertial>
   </link>
   <joint name="shoulder" type="revolute">
     <axis xyz="0 1 0"/>
-    <limit effort="18" lower="${radians(-108)}" upper="${radians(113)}" velocity="${pi}"/>
-    <origin rpy="0 0 0" xyz="0 0 0.03865"/>
-    <parent link="$(arg robot_name)/shoulder_link"/>
-    <child link="$(arg robot_name)/upper_arm_link"/>
-    <dynamics friction="0.1"/>
+    <limit
+      effort="${shoulder_limit_effort}"
+      lower="${shoulder_limit_lower}"
+      upper="${shoulder_limit_upper}"
+      velocity="${shoulder_limit_vel}"/>
+    <origin
+      rpy="0 0 0"
+      xyz="0 0 0.03865"/>
+    <parent
+      link="$(arg robot_name)/shoulder_link"/>
+    <child
+      link="$(arg robot_name)/upper_arm_link"/>
+    <dynamics
+      friction="0.1"
+      damping="0.1"/>
   </joint>
-  <transmission name="trans_shoulder">
-    <type>transmission_interface/SimpleTransmission</type>
-    <joint name="shoulder">
-      <hardwareInterface>hardware_interface/EffortJointInterface</hardwareInterface>
-    </joint>
-    <actuator name="shoulder_motor">
-      <mechanicalReduction>1</mechanicalReduction>
-    </actuator>
-  </transmission>
   <link name="$(arg robot_name)/upper_arm_link">
     <visual>
-      <origin rpy="0 0 ${pi/2}" xyz="0 0 0"/>
-      <geometry>
-        <mesh filename="package://interbotix_xsarm_descriptions/meshes/wx200_meshes/wx200_3_upper_arm.stl" scale="0.001 0.001 0.001"/>
+      <origin
+        rpy="0 0 ${pi/2}"
+        xyz="0 0 0"/>
+      <geometry>
+        <mesh
+          filename="${mesh_directory}/upper_arm.stl"
+          scale="0.001 0.001 0.001"/>
       </geometry>
       <material name="interbotix_black"/>
     </visual>
     <collision>
-      <origin rpy="0 0 ${pi/2}" xyz="0 0 0"/>
-      <geometry>
-        <mesh filename="package://interbotix_xsarm_descriptions/meshes/wx200_meshes/wx200_3_upper_arm.stl" scale="0.001 0.001 0.001"/>
+      <origin
+        rpy="0 0 ${pi/2}"
+        xyz="0 0 0"/>
+      <geometry>
+        <mesh
+          filename="${mesh_directory}/upper_arm.stl"
+          scale="0.001 0.001 0.001"/>
       </geometry>
     </collision>
     <inertial>
-      <origin rpy="0 0 ${pi/2}" xyz="0.0119707000 -0.0001179264 0.1394290000"/>
-      <mass value="0.297781" />
-      <inertia ixx="0.0017100000" iyy="0.0016310000" izz="0.0001482000" ixy="-0.0000011433" ixz="0.0000021161" iyz="0.0002135000" />
+      <origin
+        rpy="0 0 ${pi/2}"
+        xyz="0.0119707000 -0.0001179264 0.1394290000"/>
+      <mass value="0.297781"/>
+      <inertia
+        ixx="0.0017100000"
+        iyy="0.0016310000"
+        izz="0.0001482000"
+        ixy="-0.0000011433"
+        ixz="0.0000021161"
+        iyz="0.0002135000"/>
     </inertial>
   </link>
   <joint name="elbow" type="revolute">
     <axis xyz="0 1 0"/>
-    <limit effort="13" lower="${radians(-108)}" upper="${radians(93)}" velocity="${pi}"/>
-    <origin rpy="0 0 0" xyz="0.05 0 0.2"/>
-    <parent link="$(arg robot_name)/upper_arm_link"/>
-    <child link="$(arg robot_name)/forearm_link"/>
-    <dynamics friction="0.1"/>
+    <limit
+      effort="${elbow_limit_effort}"
+      lower="${elbow_limit_lower}"
+      upper="${elbow_limit_upper}"
+      velocity="${elbow_limit_vel}"/>
+    <origin
+      rpy="0 0 0"
+      xyz="0.05 0 0.2"/>
+    <parent
+      link="$(arg robot_name)/upper_arm_link"/>
+    <child
+      link="$(arg robot_name)/forearm_link"/>
+    <dynamics
+      friction="0.1"
+      damping="0.1"/>
   </joint>
-  <transmission name="trans_elbow">
-    <type>transmission_interface/SimpleTransmission</type>
-    <joint name="elbow">
-      <hardwareInterface>hardware_interface/EffortJointInterface</hardwareInterface>
-    </joint>
-    <actuator name="elbow_motor">
-      <mechanicalReduction>1</mechanicalReduction>
-    </actuator>
-  </transmission>
   <link name="$(arg robot_name)/forearm_link">
     <visual>
-      <origin rpy="0 0 ${pi/2}" xyz="0 0 0"/>
-      <geometry>
-        <mesh filename="package://interbotix_xsarm_descriptions/meshes/wx200_meshes/wx200_4_forearm.stl" scale="0.001 0.001 0.001"/>
+      <origin
+        rpy="0 0 ${pi/2}"
+        xyz="0 0 0"/>
+      <geometry>
+        <mesh
+          filename="${mesh_directory}/forearm.stl"
+          scale="0.001 0.001 0.001"/>
       </geometry>
       <material name="interbotix_black"/>
     </visual>
     <collision>
-      <origin rpy="0 0 ${pi/2}" xyz="0 0 0"/>
-      <geometry>
-        <mesh filename="package://interbotix_xsarm_descriptions/meshes/wx200_meshes/wx200_4_forearm.stl" scale="0.001 0.001 0.001"/>
+      <origin
+        rpy="0 0 ${pi/2}"
+        xyz="0 0 0"/>
+      <geometry>
+        <mesh
+          filename="${mesh_directory}/forearm.stl"
+          scale="0.001 0.001 0.001"/>
       </geometry>
     </collision>
     <inertial>
-      <origin rpy="0 0 ${pi/2}" xyz="0.1211920000 -0.0001238123 0.0000000000"/>
-      <mass value="0.283651" />
-      <inertia ixx="0.0011850000" iyy="0.0000682900" izz="0.0012060000" ixy="-0.0000024317" ixz="0.0000000000" iyz="0.0000000000" />
+      <origin
+        rpy="0 0 ${pi/2}"
+        xyz="0.1211920000 -0.0001238123 0.0000000000"/>
+      <mass value="0.283651"/>
+      <inertia
+        ixx="0.0011850000"
+        iyy="0.0000682900"
+        izz="0.0012060000"
+        ixy="-0.0000024317"
+        ixz="0.0000000000"
+        iyz="0.0000000000"/>
     </inertial>
   </link>
   <joint name="wrist_angle" type="revolute">
     <axis xyz="0 1 0"/>
-    <limit effort="5" lower="${radians(-100)}" upper="${radians(123)}" velocity="${pi}"/>
-    <origin rpy="0 0 0" xyz="0.2 0 0"/>
-    <parent link="$(arg robot_name)/forearm_link"/>
-    <child link="$(arg robot_name)/wrist_link"/>
-    <dynamics friction="0.1"/>
+    <limit
+      effort="${wrist_angle_limit_effort}"
+      lower="${wrist_angle_limit_lower}"
+      upper="${wrist_angle_limit_upper}"
+      velocity="${wrist_angle_limit_vel}"/>
+    <origin
+      rpy="0 0 0"
+      xyz="0.2 0 0"/>
+    <parent
+      link="$(arg robot_name)/forearm_link"/>
+    <child
+      link="$(arg robot_name)/wrist_link"/>
+    <dynamics
+      friction="0.1"
+      damping="0.1"/>
   </joint>
-  <transmission name="trans_wrist_angle">
-    <type>transmission_interface/SimpleTransmission</type>
-    <joint name="wrist_angle">
-      <hardwareInterface>hardware_interface/EffortJointInterface</hardwareInterface>
-    </joint>
-    <actuator name="wrist_angle_motor">
-      <mechanicalReduction>1</mechanicalReduction>
-    </actuator>
-  </transmission>
   <link name="$(arg robot_name)/wrist_link">
     <visual>
-      <origin rpy="0 0 ${pi/2}" xyz="0 0 0"/>
-      <geometry>
-        <mesh filename="package://interbotix_xsarm_descriptions/meshes/wx200_meshes/wx200_5_wrist.stl" scale="0.001 0.001 0.001"/>
+      <origin
+        rpy="0 0 ${pi/2}"
+        xyz="0 0 0"/>
+      <geometry>
+        <mesh
+          filename="${mesh_directory}/wrist.stl"
+          scale="0.001 0.001 0.001"/>
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