Commit message: Refactor gripper controller and modes for PWM operation - Updated controller configuration to use gripper_pwm_bridge instead of gripper_controller. - Changed gripper operating mode to PWM in modes.yaml. - Adjusted grasping and released joint values in wx200.srdf.xacro. - Modified xsarm_moveit.launch.py to include move_group capabilities. - Commented out redundant gripper command publishing in xs_hardware_interface.cpp.

File: interbotix_ros_manipulators/interbotix_ros_xsarms/interbotix_xsarm_moveit/config/srdf/wx200.srdf.xacro (robot description, xacro)
@@ -53,10 +53,10 @@
     </group_state>
     <group_state name="Grasping" group="interbotix_gripper">
-        <joint name="left_finger" value="0.015" />
-        <joint name="right_finger" value="-0.015" />
+        <joint name="left_finger" value="0.017" />
+        <joint name="right_finger" value="-0.017" />
     </group_state>
     <group_state name="Released" group="interbotix_gripper">
-        <joint name="left_finger" value="0.037" />
-        <joint name="right_finger" value="-0.037" />
+        <joint name="left_finger" value="0.030" />
+        <joint name="right_finger" value="-0.030" />
     </group_state>
     <group_state name="Home" group="interbotix_gripper">
